File: hw/main_part/hackeriet_imponator/hackeriet_imponator.kicad_pcb (KiCad board)
At the start: 2 copper layers, 118.1 x 118.1 mm, 8 parts, among them U1 ATmega328PB-A

Commit message: Added ring. Added programming header. Started with batt connector
Parts:
- added D5: WS2812B, LED_SMD:LED_WS2812B_PLCC4_5.0x5.0mm_P3.2mm, B.Cu at (56.0, 142.8)
- added D6: WS2812B, LED_SMD:LED_WS2812B_PLCC4_5.0x5.0mm_P3.2mm, B.Cu at (-9.65, 113.5)
- added H10: MountingHole_Pad, MountingHole:MountingHole_3.2mm_M3_Pad_Via, F.Cu at (94.0, 91.0)
- added H11: MountingHole_Pad, MountingHole:MountingHole_3.2mm_M3_Pad_Via, F.Cu at (40.0, 145.0)
- added H12: MountingHole_Pad, MountingHole:MountingHole_3.2mm_M3_Pad_Via, F.Cu at (40.0, 37.0)
- added H9: MountingHole_Pad, MountingHole:MountingHole_3.2mm_M3_Pad_Via, F.Cu at (-14.0, 91.0)
- added J1: AVR-ISP-6, Connector_PinSocket_2.54mm:PinSocket_2x03_P2.54mm_Vertical_SMD, B.Cu at (180.2, 44.0)
- added J2: Battery connector, imponator_footprint_lib:BAT_1022, F.Cu at (297.5, 47.5)
- moved H3 21.1 mm to (179.5, 138.5)
- moved H2 21.0 mm to (233.5, 84.5)
- moved H1 20.9 mm to (125.5, 84.5)
- moved H4 20.8 mm to (179.5, 30.5)
Connections:
- U1 pad 15: unconnected-(U1-PB3-Pad15) -> Net-(J1-MOSI)
- U1 pad 16: unconnected-(U1-PB4-Pad16) -> Net-(J1-MISO)
- U1 pad 17: unconnected-(U1-PB5-Pad17) -> Net-(J1-SCK)
- U1 pad 29: unconnected-(U1-~{RESET}/PC6-Pad29) -> Net-(J1-~{RST})
Routing:
- net +3.3V: track 106.5 -> 215.6 mm
- net Net-(D5-DOUT): track 0.00 -> 73.6 mm
- net Net-(D5-DIN): track 0.00 -> 67.1 mm
- net Net-(D2-DOUT): track 39.3 -> 23.8 mm
- net Net-(J2-Pin_2): track 0.00 -> 10.9 mm
- net GND: track 5.14 -> 3.77 mm
- net (no net): track 0.00 -> 1.00 mm
Other:
- board size 118.1 x 118.1 mm -> 257.6 x 124.6 mm
