File: hw/hackeriet_imponator/hackeriet_imponator.kicad_sch (KiCad schematic)
At the start: 34 parts, among them J1 USB4085-GF-A, J2 UPDI programming, J3 External Battery Connector, J4 Shitty Add On, J5 Unused pins, SW1 SW_SPDT, SW2 User configurable, SW3 User configurable, U1 ATtiny804-SS, U2 MCP2221AxSL, U3 MPU-6050, U4 TLV70028_SOT353

Commit message: Did a bunch of routing and changed holes. Also some silk
Parts:
- added C9: 100nF, Capacitor_SMD:C_0603_1608Metric_Pad1.08x0.95mm_HandSolder, symbol Device:C
Connections:
- net WS2812B LED RGB Control plate is gone; now on net WS2812B LED RGB Control logo: U1.11 (PA1)
- net GND: now also C9.2
- net VDD: now also C9.1
- net WS2812B LED RGB Control renamed WS2812B LED RGB Control logo
Other:
- moved on the sheet: C2
Changed lines of the file:
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@@
 	)
 	(junction
+		(at 125.73 107.95)
+		(diameter 0)
+		(color 0 0 0 0)
+	)
+	(junction
 		(at 187.96 137.16)
 		(diameter 0)
@@
 	)
 	(junction
+		(at 106.68 101.6)
+		(diameter 0)
+		(color 0 0 0 0)
+	)
+	(junction
 		(at 160.02 130.81)
 		(diameter 0)
@@
 	(wire
 		(pts
-			(xy 109.22 106.68) (xy 109.22 109.22)
+			(xy 160.02 130.81) (xy 160.02 135.89)
 		)
 		(stroke
@@
 	(wire
 		(pts
-			(xy 160.02 130.81) (xy 160.02 135.89)
+			(xy 121.92 64.77) (xy 124.46 64.77)
 		)
 		(stroke
@@
 	(wire
 		(pts
-			(xy 121.92 64.77) (xy 124.46 64.77)
+			(xy 123.19 107.95) (xy 125.73 107.95)
 		)
 		(stroke
@@
 	(wire
 		(pts
-			(xy 116.84 106.68) (xy 119.38 106.68)
+			(xy 59.69 116.84) (xy 62.23 116.84)
 		)
 		(stroke
@@
 	(wire
 		(pts
-			(xy 59.69 116.84) (xy 62.23 116.84)
+			(xy 125.73 101.6) (xy 116.84 101.6)
 		)
 		(stroke
@@
 	(wire
 		(pts
+			(xy 125.73 107.95) (xy 125.73 101.6)
+		)
+		(stroke
+			(width 0)
+			(type default)
+		)
+	)
+	(wire
+		(pts
 			(xy 109.22 58.42) (xy 109.22 64.77)
 		)
@@
 	(wire
 		(pts
+			(xy 106.68 101.6) (xy 106.68 109.22)
+		)
+		(stroke
+			(width 0)
+			(type default)
+		)
+	)
+	(wire
+		(pts
 			(xy 59.69 127) (xy 66.04 127)
 		)
@@
 	(wire
 		(pts
+			(xy 109.22 101.6) (xy 106.68 101.6)
+		)
+		(stroke
+			(width 0)
+			(type default)
+		)
+	)
+	(wire
+		(pts
 			(xy 181.61 60.96) (xy 176.53 60.96)
 		)
@@
 	(wire
 		(pts
-			(xy 175.26 27.94) (xy 151.13 27.94)
+			(xy 181.61 27.94) (xy 151.13 27.94)
+		)
+		(stroke
+			(width 0)
+			(type default)
+		)
+	)
+	(wire
+		(pts
+			(xy 115.57 107.95) (xy 109.22 107.95)
 		)
 		(stroke
@@
 	(wire
 		(pts
+			(xy 109.22 107.95) (xy 109.22 109.22)
+		)
+		(stroke
+			(width 0)
+			(type default)
+		)
+	)
+	(wire
+		(pts
 			(xy 152.4 110.49) (xy 160.02 110.49)
 		)
@@
 	(wire
 		(pts
-			(xy 175.26 25.4) (xy 175.26 27.94)
+			(xy 181.61 25.4) (xy 181.61 27.94)
 		)
 		(stroke
@@
 		)
 	)
-	(global_label "WS2812B LED RGB Control"
+	(global_label "PA5"
 		(shape input)
-		(at 175.26 25.4 180)
+		(at 81.28 60.96 0)
 		(fields_autoplaced yes)
 		(effects
@@
 				(size 1.27 1.27)
 			)
-			(justify right)
+			(justify left)
 		)
 		(property "Intersheetrefs" "${INTERSHEET_REFS}"
-			(at 146.4519 25.4 0)
+			(at 87.8333 60.96 0)
 			(effects
 				(font
 					(size 1.27 1.27)
 				)
-				(justify right)
+				(justify left)
 				(hide yes)
 			)
 		)
 	)
-	(global_label "PA5"
+	(global_label "WS2812B LED RGB Control logo"
 		(shape input)
-		(at 81.28 60.96 0)
+		(at 86.36 50.8 0)
 		(fields_autoplaced yes)
 		(effects
@@
 		)
 		(property "Intersheetrefs" "${INTERSHEET_REFS}"
-			(at 87.8333 60.96 0)
+			(at 120.2479 50.8 0)
 			(effects
 				(font
@@
 		)
 	)
-	(global_label "WS2812B LED RGB Control plate"
+	(global_label "MCP2221 _RST"
 		(shape input)
-		(at 86.36 50.8 0)
+		(at 81.28 66.04 0)
 		(fields_autoplaced yes)
 		(effects
@@
 		)
 		(property "Intersheetrefs" "${INTERSHEET_REFS}"
-			(at 120.9132 50.8 0)
+			(at 98.4769 66.04 0)
 			(effects
 				(font
@@
 		)
 	)
-	(global_label "MCP2221 _RST"
+	(global_label "SCL"
 		(shape input)
-		(at 81.28 66.04 0)
+		(at 39.37 48.26 180)
 		(fields_autoplaced yes)
 		(effects
@@
 				(size 1.27 1.27)
 			)
-			(justify left)
+			(justify right)
 		)
 		(property "Intersheetrefs" "${INTERSHEET_REFS}"
-			(at 98.4769 66.04 0)
+			(at 32.8772 48.26 0)
 			(effects
 				(font
 					(size 1.27 1.27)
 				)
-				(justify left)
+				(justify right)
 				(hide yes)
 			)
 		)
 	)
-	(global_label "SCL"
+	(global_label "D+"
 		(shape input)
-		(at 39.37 48.26 180)
+		(at 78.74 123.19 180)
 		(fields_autoplaced yes)
 		(effects
@@
 		)
 		(property "Intersheetrefs" "${INTERSHEET_REFS}"
-			(at 32.8772 48.26 0)
+			(at 72.9124 123.19 0)
 			(effects
 				(font
@@
 		)
 	)
-	(global_label "D+"
+	(global_label "WS2812B LED RGB Control logo"
 		(shape input)
-		(at 78.74 123.19 180)
+		(at 181.61 25.4 180)
 		(fields_autoplaced yes)
 		(effects
@@
 		)
 		(property "Intersheetrefs" "${INTERSHEET_REFS}"
-			(at 72.9124 123.19 0)
+			(at 147.7221 25.4 0)
 			(effects
 				(font
@@
 	(symbol
 		(lib_id "Device:C")
-		(at 113.03 106.68 90)
+		(at 119.38 107.95 90)
 		(unit 1)
 		(exclude_from_sim no)
@@
 		(dnp no)
 		(property "Reference" "C2"
-			(at 113.03 103.124 90)
+			(at 119.38 104.394 90)
 			(effects
 				(font
@@
 		)
 		(property "Value" "1uF"
-			(at 113.03 109.982 90)
+			(at 119.38 111.252 90)
 			(effects
 				(font
@@
 		)
 		(property "Footprint" "Capacitor_SMD:C_0603_1608Metric_Pad1.08x0.95mm_HandSolder"
-			(at 116.84 105.7148 0)
+			(at 123.19 106.9848 0)
 			(effects
 				(font
@@
 		)
 		(property "Datasheet" "~"
-			(at 113.03 106.68 0)
+			(at 119.38 107.95 0)
 			(effects
 				(font
@@
 		)
 		(property "Description" "Unpolarized capacitor"
-			(at 113.03 106.68 0)
+			(at 119.38 107.95 0)
 			(effects
 				(font
@@
 	)
 	(symbol
+		(lib_id "Device:C")
+		(at 113.03 101.6 90)
+		(unit 1)
+		(exclude_from_sim no)
+		(in_bom yes)
+		(on_board yes)
+		(dnp no)
+		(property "Reference" "C9"
+			(at 115.824 98.552 90)
+			(effects
+				(font
+					(size 1.27 1.27)
+				)
+			)
+		)
+		(property "Value" "100nF"
+			(at 113.538 104.902 90)
+			(effects
+				(font
+					(size 1.27 1.27)
+				)
+			)
+		)
+		(property "Footprint" "Capacitor_SMD:C_0603_1608Metric_Pad1.08x0.95mm_HandSolder"
+			(at 116.84 100.6348 0)
+			(effects
+				(font
+					(size 1.27 1.27)
+				)
+				(hide yes)
+			)
+		)
+		(property "Datasheet" "~"
+			(at 113.03 101.6 0)
+			(effects
+				(font
+					(size 1.27 1.27)
+				)
+				(hide yes)
+			)
+		)
+		(property "Description" "Unpolarized capacitor"
+			(at 113.03 101.6 0)
+			(effects
+				(font
+					(size 1.27 1.27)
+				)
+				(hide yes)
+			)
+		)
+		(pin "2"
+		)
+		(pin "1"
+		)
+		(instances
+			(project "hackeriet_imponator"
+				(path "/469a2550-d397-4ef7-965d-96f8e6eb26aa"
+					(reference "C9")
+					(unit 1)
+				)
+			)
+		)
+	)
+	(symbol
 		(lib_id "power:GND")
 		(at 58.42 36.83 0)
@@
 	(symbol
 		(lib_id "power:GND")
-		(at 119.38 106.68 0)
+		(at 125.73 107.95 0)
 		(mirror y)
 		(unit 1)
@@
 		(dnp no)
 		(property "Reference" "#PWR016"
-			(at 119.38 113.03 0)
+			(at 125.73 114.3 0)
 			(effects
 				(font
@@
 		)
 		(property "Value" "GND"
-			(at 121.666 109.982 0)
+			(at 128.016 111.252 0)
 			(effects
 				(font
@@
 		)
 		(property "Footprint" ""
-			(at 119.38 106.68 0)
+			(at 125.73 107.95 0)
 			(effects
 				(font
@@
 		)
 		(property "Datasheet" ""
-			(at 119.38 106.68 0)
+			(at 125.73 107.95 0)
 			(effects
 				(font
@@
 		)
 		(property "Description" "Power symbol creates a global label with name \"GND\" , ground"
-			(at 119.38 106.68 0)
+			(at 125.73 107.95 0)
 			(effects
 				(font
@@
 	(symbol
 		(lib_id "power:+3.3V")
-		(at 106.68 109.22 0)
+		(at 106.68 101.6 0)
 		(unit 1)
 		(exclude_from_sim no)
@@
 		(dnp no)
 		(property "Reference" "#PWR014"
-			(at 106.68 113.03 0)
+			(at 106.68 105.41 0)
 			(effects
 				(font
@@
 		)
 		(property "Value" "VDD"
-			(at 105.918 105.156 0)
+			(at 108.966 99.06 0)
 			(effects
 				(font
@@
 		)
 		(property "Footprint" ""
-			(at 106.68 109.22 0)
+			(at 106.68 101.6 0)
 			(effects
 				(font
@@
 		)
 		(property "Datasheet" ""
-			(at 106.68 109.22 0)
+			(at 106.68 101.6 0)
 			(effects
 				(font
@@
 		)
 		(property "Description" "Power symbol creates a global label with name \"+3.3V\""
-			(at 106.68 109.22 0)
+			(at 106.68 101.6 0)
 			(effects
 				(font
